Commit message: Arm and camera added

File: rover_description/urdf/rover.xacro (robot description, xacro)
@@ -2,27 +2,47 @@
 <robot name="rover" xmlns:xacro="http://www.ros.org/wiki/xacro">
   <xacro:property name="PI" value="3.1415926535897931"/>
-  <xacro:property name="chassisHeight" value="0.25"/>
-  <xacro:property name="chassisLength" value="0.6"/>
+  <xacro:property name="chassisHeight" value="0.3"/>
+  <xacro:property name="chassisLength" value="0.75"/>
   <xacro:property name="chassisWidth" value="0.45"/>
   <xacro:property name="chassisMass" value="50"/>
-  <xacro:property name="casterRadius" value="0.05"/>
-  <xacro:property name="casterMass" value="5"/>
-  <xacro:property name="wheelWidth" value="0.06"/>
-  <xacro:property name="wheelRadius" value="0.1"/>
-  <xacro:property name="wheelPos" value="0.2"/>
+  <!--stick out 0.285 wheel drop = 0.12-->
+  <xacro:property name="wheelWidth" value="0.075"/>
+  <xacro:property name="wheelRadius" value="0.21"/>
+  <xacro:property name="wheelPos" value="0.3"/>
   <xacro:property name="wheelMass" value="5"/>
   <xacro:property name="cameraSize" value="0.05"/>
   <xacro:property name="cameraMass" value="0.1"/>
+  <xacro:property name="link_name" value="depth"/>
+  <xacro:property name="frame_name" value="camera_link"/>
+  <xacro:property name="camera_name" value="camera"/>
   <xacro:include filename="$(find rover_description)/urdf/rover.gazebo"/>
   <xacro:include filename="$(find rover_description)/urdf/materials.xacro"/>
   <xacro:include filename="$(find rover_description)/urdf/macros.xacro"/>
-  <link name="base_link"/>
-  <joint name="base_joint" type="fixed">
-    <parent link="base_link"/>
-    <child link="chassis"/>
-  </joint>
-  <link name="chassis">
-    <collision>
-      <origin xyz="0 0 ${wheelRadius}" rpy="0 0 0"/>
+  <!--xacro:include filename="$(find rover_description)/urdf/arm.xacro"/-->
+  <xacro:property name="PI" value="3.1415926535897931"/>
+  <xacro:property name="plateLength" value="0.180"/>
+  <xacro:property name="plateWidth" value="0.25"/>
+  <xacro:property name="plateMass" value="0.267"/>
+  <xacro:property name="plateHeight" value="0.006"/>
+  <xacro:property name="baseHeight" value="0.0635"/>
+  <xacro:property name="baseRadius" value="0.12"/>
+  <xacro:property name="motor2Length" value="0.36"/>
+  <xacro:property name="motor3Length" value="0.5"/>
+  <xacro:property name="chassisWidth" value="0.45"/>
+  <xacro:property name="baseDamping" value="0.1"/>
+  <xacro:property name="sidePlateLenght" value="0.25"/>
+  <xacro:property name="sidePlateWidth" value="0.05"/>
+  <xacro:property name="sidePlateHeight" value="0.165"/>
+  <xacro:property name="motor2Length" value="0.36"/>
+  <xacro:property name="motor2Radius" value="0.08"/>
+  <xacro:property name="sidePlate2Motor2Damping" value="0.1"/>
+  <xacro:property name="motor3Length" value="0.5"/>
+  <xacro:property name="motor3Radius" value="0.05"/>
+  <xacro:property name="excavatorLenght" value="0.005"/>
+  <xacro:property name="excavatorWidth" value="0.078"/>
+  <xacro:property name="excavatorHeight" value="0.078"/>
+  <link name="base_link">
+    <collision>
+      <origin xyz="0 0 0" rpy="0 0 0"/>
       <geometry>
         <box size="${chassisLength} ${chassisWidth} ${chassisHeight}"/>
@@ -30,12 +50,12 @@
     </collision>
     <visual>
-      <origin xyz="0 0 ${wheelRadius}" rpy="0 0 0"/>
+      <origin xyz="0 0 0" rpy="0 0 0"/>
       <geometry>
         <box size="${chassisLength} ${chassisWidth} ${chassisHeight}"/>
       </geometry>
-      <material name="orange"/>
-    </visual>
-    <inertial>
-      <origin xyz="0 0 ${wheelRadius}" rpy="0 0 0"/>
+      <material name="green"/>
+    </visual>
+    <inertial>
+      <origin xyz="0 0 0" rpy="0 0 0"/>
       <mass value="${chassisMass}"/>
       <box_inertia m="${chassisMass}" x="${chassisLength}" y="${chassisWidth}" z="${chassisHeight}"/>
@@ -47,51 +67,163 @@
   <wheel lr="back_right" tY="-1" tX="-1"/>
   <joint name="camera_joint" type="fixed">
-    <origin xyz="${-cameraSize+chassisLength/2} 0 ${cameraSize+wheelRadius+cameraSize/2}" rpy="0 0 0"/>
-    <parent link="chassis"/>
-    <child link="camera"/>
-  </joint>
-  <link name="camera">
-    <collision>
-      <origin xyz="0 0 0" rpy="0 0 0"/>
-      <geometry>
-        <box size="${cameraSize} ${cameraSize} ${cameraSize}"/>
-      </geometry>
-    </collision>
-    <visual>
-      <origin xyz="0 0 0" rpy="0 0 0"/>
-      <geometry>
-        <box size="${cameraSize} ${cameraSize} ${cameraSize}"/>
+    <axis xyz="0 0 0"/>
+    <parent link="base_link"/>
+    <child link="camera_link"/>
+    <origin xyz="${chassisLength/2} 0 ${chassisHeight/2}" rpy="0 0 0"/>
+  </joint>
+  <link name="camera_link">
+    <collision>
+      <origin xyz="0 0 0.025" rpy="0 0 0"/>
+      <geometry>
+        <box size="0.05 0.1 0.05"/>
+      </geometry>
+    </collision>
+    <visual>
+      <origin xyz="0 0 0.025" rpy="0 0 0"/>
+      <geometry>
+        <box size="0.05 0.1 0.05"/>
       </geometry>
       <material name="blue"/>
     </visual>
     <inertial>
-      <mass value="${cameraMass}"/>
-      <origin xyz="0 0 0" rpy="0 0 0"/>
-      <box_inertia m="${cameraMass}" x="${cameraSize}" y="${cameraSize}" z="${cameraSize}"/>
-    </inertial>
-  </link>
-  <!--joint name="fixed" type="fixed">
-  <parent link="chassis"/>
-  <child link="caster_wheel"/>
-</joint>
-s
-<link name="caster_wheel">
-<collision>
-<origin xyz="${casterRadius-chassisLength/2} 0 ${casterRadius-chassisHeight+wheelRadius}" rpy="0 0 0"/>
-<geometry>
-<sphere radius="${casterRadius}"/>
-</geometry>
-</collision>
-<visual>
-<origin xyz="${casterRadius-chassisLength/2} 0 ${casterRadius-chassisHeight+wheelRadius}" rpy="0 0 0"/>
-<geometry>
-<sphere radius="${casterRadius}"/>
-</geometry>
-</visual>
-<inertial>
-<origin xyz="${casterRadius-chassisLength/2} 0 ${casterRadius-chassisHeight+wheelRadius}" rpy="0 0 0"/>
-<mass value="${casterMass}"/>
-<sphere_inertia m="${casterMass}" r="${casterRadius}"/>
-</inertial>
-</link-->
+      <mass value="1e-5"/>
+      <origin xyz="0 0 0.025" rpy="0 0 0"/>
+      <inertia ixx="1e-6" ixy="0" ixz="0" iyy="1e-6" iyz="0" izz="1e-6"/>
+    </inertial>
+  </link>
+  <joint name="arm_base_joint" type="revolute">
+    <axis xyz="0 0 1"/>
+    <parent link="base_link"/>
+    <child link="arm_base_link"/>
+    <limit lower="-90" upper="90" effort="1" velocity="2"/>
+    <origin xyz="0 0 ${chassisHeight/2}" rpy="0 0 0"/>
+  </joint>
+  <link name="arm_base_link">
+    <visual>
+      <origin xyz="0 0 ${baseHeight/2}" rpy="0 0 0"/>
+      <geometry>
+        <cylinder length="${baseHeight}" radius="${baseRadius}"/>
+      </geometry>
+    </visual>
+    <inertial>
+      <mass value="${wheelMass}"/>
+      <origin xyz="0 0 ${baseHeight/2}" rpy="0 0 0"/>
+      <cylinder_inertia m="${wheelMass}" r="${wheelRadius}" h="${wheelWidth}"/>
+    </inertial>
+    <collision>
+      <origin xyz="0 0 ${baseHeight/2}" rpy="0 0 0"/>
+      <geometry>
+        <cylinder length="${baseHeight}" radius="${baseRadius}"/>
+      </geometry>
+    </collision>
+  </link>
+  <joint name="joint_base_side_plate" type="fixed">
+    <parent link="arm_base_link"/>
+    <child link="side_plate"/>
+    <origin xyz="0 0 ${baseHeight}" rpy="0 0 0"/>
+  </joint>
+  <link name="side_plate">
+    <inertial>
+      <origin xyz="0 0 0" rpy="0 0 0"/>
+      <mass value="0.130"/>
+      <inertia ixx="1837000" ixy="120300" ixz="279500" iyy="1651000" iyz="620400" izz="34900"/>
+    </inertial>
+    <visual>
+      <origin xyz="0 0 ${sidePlateHeight/2}" rpy="0 0 0"/>
+      <geometry>
+        <box size="${sidePlateLenght} ${sidePlateWidth} ${sidePlateHeight}"/>
+      </geometry>
+      <material name="black"/>
+    </visual>
+    <collision>
+      <origin xyz="0 0 ${sidePlateHeight/2}" rpy="0 0 0"/>
+      <geometry>
+        <box size="${sidePlateLenght} ${sidePlateWidth} ${sidePlateHeight}"/>
+      </geometry>
+    </collision>
+  </link>
+  <joint name="side_motor2" type="revolute">
+    <parent link="side_plate"/>
+    <child link="motor2"/>
+    <axis xyz=" 0 1 0"/>
+    <origin xyz="0 0  ${sidePlateHeight}" rpy="0 0 0"/>
+    <dynamics damping="${sidePlate2Motor2Damping}"/>
+    <limit effort="100.0" velocity="0.5" lower="-1.571" upper="1.571"/>
+  </joint>
+  <link name="motor2">
+    <visual>
+      <origin xyz="0 0 ${motor2Length/2}" rpy="0 0 0"/>
+      <material name="black"/>
+      <geometry>
+        <cylinder length="${motor2Length}" radius="${motor2Radius}"/>
+      </geometry>
+    </visual>
+    <collision>
+      <origin xyz="0 0 ${motor2Length/2}" rpy="0 0 0"/>
+      <geometry>
+        <cylinder length="${motor2Length}" radius="${motor2Radius}"/>
+      </geometry>
+    </collision>
+    <inertial>
+      <origin xyz="0.416 0 0.154" rpy="0 0 0"/>
+      <mass value="2"/>
+      <inertia ixx="1940000" ixy="0" ixz="-1620000" iyy="3217000" iyz="0" izz="1940000"/>
+    </inertial>
+  </link>
+  <joint name="motor2_motor3_joint" type="revolute">
+    <parent link="motor2"/>
+    <child link="motor3"/>
+    <axis xyz=" 0 1 0"/>
+    <origin xyz="0 0 ${motor2Length}" rpy="0 0 0"/>
+    <dynamics damping="${sidePlate2Motor2Damping}"/>
+    <limit effort="100.0" velocity="0.5" lower="-1.571" upper="1.571"/>
+  </joint>
+  <link name="motor3">
+    <visual>
+      <origin xyz="0 0 ${motor3Length/2}" rpy="0 0 0"/>
+      <material name="black"/>
+      <geometry>
+        <cylinder length="${motor3Length}" radius="${motor3Radius}"/>
+      </geometry>
+    </visual>
+    <collision>
+      <origin xyz="0 0 ${motor3Length/2}" rpy="0 0 0"/>
+      <geometry>
+        <cylinder length="${motor3Length}" radius="${motor3Radius}"/>
+      </geometry>
+    </collision>
+    <inertial>
+      <origin xyz="0.5 0 0.5" rpy="0 0 0"/>
+      <mass value="1"/>
+      <inertia ixx="57630000" ixy="0" ixz="-50390000" iyy="116300000" iyz="0" izz="59050000"/>
+    </inertial>
+  </link>
+  <joint name="motor3_end_effector_joint" type="revolute">
+    <parent link="motor3"/>
+    <child link="end_effector"/>
+    <axis xyz=" 0 1 0"/>
+    <origin xyz="0 0 ${motor3Length}" rpy="0 0 0"/>
+    <dynamics damping="${sidePlate2Motor2Damping}"/>
+    <limit effort="100.0" velocity="0.5" lower="-1.571" upper="1.571"/>
+  </joint>
+  <link name="end_effector">
+    <inertial>
+      <origin xyz="0 0 1.0945" rpy="0 0 0"/>
+      <mass value="0.1"/>
+      <inertia ixx="13410" ixy="0.0" ixz="0.0" iyy="13850" iyz="0.0" izz="27150"/>
+    </inertial>
+    <visual>
+      <origin xyz="0 0 ${excavatorHeight/2}" rpy="0 0 0"/>
+      <geometry>
+        <box size="${excavatorLenght} ${excavatorWidth} ${excavatorHeight}"/>
+      </geometry>
+      <material name="black"/>
+    </visual>
+    <collision>
+      <origin xyz="0 0 ${excavatorHeight/2}" rpy="0 0 0"/>
+      <geometry>
+        <box size="${excavatorLenght} ${excavatorWidth} ${excavatorHeight}"/>
+      </geometry>
+    </collision>
+  </link>
 </robot>

Commit message: Fixed wrong arm links inertias

File: rover_description/urdf/rover.xacro (robot description, xacro)
@@ -8,7 +8,8 @@
   <!--stick out 0.285 wheel drop = 0.12-->
   <xacro:property name="wheelWidth" value="0.075"/>
-  <xacro:property name="wheelRadius" value="0.21"/>
+  <xacro:property name="wheelRadius" value="0.18"/>
   <xacro:property name="wheelPos" value="0.3"/>
   <xacro:property name="wheelMass" value="5"/>
+  <xacro:property name="wheelDrop" value="-0.12"/>
   <xacro:property name="cameraSize" value="0.05"/>
   <xacro:property name="cameraMass" value="0.1"/>
@@ -20,5 +21,4 @@
   <xacro:include filename="$(find rover_description)/urdf/macros.xacro"/>
   <!--xacro:include filename="$(find rover_description)/urdf/arm.xacro"/-->
-  <xacro:property name="PI" value="3.1415926535897931"/>
   <xacro:property name="plateLength" value="0.180"/>
   <xacro:property name="plateWidth" value="0.25"/>
@@ -27,6 +27,6 @@
   <xacro:property name="baseHeight" value="0.0635"/>
   <xacro:property name="baseRadius" value="0.12"/>
-  <xacro:property name="motor2Length" value="0.36"/>
-  <xacro:property name="motor3Length" value="0.5"/>
+  <xacro:property name="arm_link_1Length" value="0.36"/>
+  <xacro:property name="arm_link_2Length" value="0.5"/>
   <xacro:property name="chassisWidth" value="0.45"/>
   <xacro:property name="baseDamping" value="0.1"/>
@@ -34,9 +34,9 @@
   <xacro:property name="sidePlateWidth" value="0.05"/>
   <xacro:property name="sidePlateHeight" value="0.165"/>
-  <xacro:property name="motor2Length" value="0.36"/>
-  <xacro:property name="motor2Radius" value="0.08"/>
-  <xacro:property name="sidePlate2Motor2Damping" value="0.1"/>
-  <xacro:property name="motor3Length" value="0.5"/>
-  <xacro:property name="motor3Radius" value="0.05"/>
+  <xacro:property name="arm_link_1Length" value="0.36"/>
+  <xacro:property name="arm_link_1Radius" value="0.08"/>
+  <xacro:property name="sidePlate2arm_link_1Damping" value="0.1"/>
+  <xacro:property name="arm_link_2Length" value="0.5"/>
+  <xacro:property name="arm_link_2Radius" value="0.05"/>
   <xacro:property name="excavatorLenght" value="0.005"/>
   <xacro:property name="excavatorWidth" value="0.078"/>
@@ -92,9 +92,9 @@
     </inertial>
   </link>
-  <joint name="arm_base_joint" type="revolute">
+  <joint name="arm_joint_0" type="revolute">
     <axis xyz="0 0 1"/>
     <parent link="base_link"/>
     <child link="arm_base_link"/>
-    <limit lower="-90" upper="90" effort="1" velocity="2"/>
+    <limit lower="-2" upper="2" effort="1" velocity="2"/>
     <origin xyz="0 0 ${chassisHeight/2}" rpy="0 0 0"/>
   </joint>
@@ -127,5 +127,6 @@
       <origin xyz="0 0 0" rpy="0 0 0"/>
       <mass value="0.130"/>
-      <inertia ixx="1837000" ixy="120300" ixz="279500" iyy="1651000" iyz="620400" izz="34900"/>
+      <!--box_inertia m="0.130" x="${sidePlateLenght}" y="${sidePlateWidth}" z="${sidePlateHeight}"/-->
+      <box_inertia m="0.130" x="${sidePlateLenght}" y="${sidePlateWidth}" z="${sidePlateHeight}"/>
     </inertial>
     <visual>
@@ -143,24 +144,24 @@
     </collision>
   </link>
-  <joint name="side_motor2" type="revolute">
+  <joint name="arm_joint_1" type="revolute">
     <parent link="side_plate"/>
-    <child link="motor2"/>
+    <child link="arm_link_1"/>
     <axis xyz=" 0 1 0"/>
     <origin xyz="0 0  ${sidePlateHeight}" rpy="0 0 0"/>
-    <dynamics damping="${sidePlate2Motor2Damping}"/>
+    <dynamics damping="${sidePlate2arm_link_1Damping}"/>
     <limit effort="100.0" velocity="0.5" lower="-1.571" upper="1.571"/>
   </joint>
-  <link name="motor2">
-    <visual>
-      <origin xyz="0 0 ${motor2Length/2}" rpy="0 0 0"/>
-      <material name="black"/>
-      <geometry>
-        <cylinder length="${motor2Length}" radius="${motor2Radius}"/>
-      </geometry>
-    </visual>
-    <collision>
-      <origin xyz="0 0 ${motor2Length/2}" rpy="0 0 0"/>
-      <geometry>
-        <cylinder length="${motor2Length}" radius="${motor2Radius}"/>
+  <link name="arm_link_1">
+    <visual>
+      <origin xyz="0 0 ${arm_link_1Length/2}" rpy="0 0 0"/>
+      <material name="black"/>
+      <geometry>
+        <cylinder length="${arm_link_1Length}" radius="${arm_link_1Radius}"/>
+      </geometry>
+    </visual>
+    <collision>
+      <origin xyz="0 0 ${arm_link_1Length/2}" rpy="0 0 0"/>
+      <geometry>
+        <cylinder length="${arm_link_1Length}" radius="${arm_link_1Radius}"/>
       </geometry>
     </collision>
@@ -168,27 +169,27 @@
       <origin xyz="0.416 0 0.154" rpy="0 0 0"/>
       <mass value="2"/>
-      <inertia ixx="1940000" ixy="0" ixz="-1620000" iyy="3217000" iyz="0" izz="1940000"/>
-    </inertial>
-  </link>
-  <joint name="motor2_motor3_joint" type="revolute">
-    <parent link="motor2"/>
-    <child link="motor3"/>
+      <cylinder_inertia m="2" r="${arm_link_1Radius}" h="${arm_link_1Length}"/>
+    </inertial>
+  </link>
+  <joint name="arm_joint_2" type="revolute">
+    <parent link="arm_link_1"/>
+    <child link="arm_link_2"/>
     <axis xyz=" 0 1 0"/>
-    <origin xyz="0 0 ${motor2Length}" rpy="0 0 0"/>
-    <dynamics damping="${sidePlate2Motor2Damping}"/>
+    <origin xyz="0 0 ${arm_link_1Length}" rpy="0 0 0"/>
+    <dynamics damping="${sidePlate2arm_link_1Damping}"/>
     <limit effort="100.0" velocity="0.5" lower="-1.571" upper="1.571"/>
   </joint>
-  <link name="motor3">
-    <visual>
-      <origin xyz="0 0 ${motor3Length/2}" rpy="0 0 0"/>
-      <material name="black"/>
-      <geometry>
-        <cylinder length="${motor3Length}" radius="${motor3Radius}"/>
-      </geometry>
-    </visual>
-    <collision>
-      <origin xyz="0 0 ${motor3Length/2}" rpy="0 0 0"/>
-      <geometry>
-        <cylinder length="${motor3Length}" radius="${motor3Radius}"/>
+  <link name="arm_link_2">
+    <visual>
+      <origin xyz="0 0 ${arm_link_2Length/2}" rpy="0 0 0"/>
+      <material name="black"/>
+      <geometry>
+        <cylinder length="${arm_link_2Length}" radius="${arm_link_2Radius}"/>
+      </geometry>
+    </visual>
+    <collision>
+      <origin xyz="0 0 ${arm_link_2Length/2}" rpy="0 0 0"/>
+      <geometry>
+        <cylinder length="${arm_link_2Length}" radius="${arm_link_2Radius}"/>
       </geometry>
     </collision>
@@ -196,13 +197,13 @@
       <origin xyz="0.5 0 0.5" rpy="0 0 0"/>
       <mass value="1"/>
-      <inertia ixx="57630000" ixy="0" ixz="-50390000" iyy="116300000" iyz="0" izz="59050000"/>
-    </inertial>
-  </link>
-  <joint name="motor3_end_effector_joint" type="revolute">
-    <parent link="motor3"/>
+      <cylinder_inertia m="1" r="${arm_link_2Radius}" h="${arm_link_2Length}"/>
+    </inertial>
+  </link>
+  <joint name="arm_joint_3" type="revolute">
+    <parent link="arm_link_2"/>
     <child link="end_effector"/>
     <axis xyz=" 0 1 0"/>
-    <origin xyz="0 0 ${motor3Length}" rpy="0 0 0"/>
-    <dynamics damping="${sidePlate2Motor2Damping}"/>
+    <origin xyz="0 0 ${arm_link_2Length}" rpy="0 0 0"/>
+    <dynamics damping="${sidePlate2arm_link_1Damping}"/>
     <limit effort="100.0" velocity="0.5" lower="-1.571" upper="1.571"/>
   </joint>
@@ -211,5 +212,5 @@
       <origin xyz="0 0 1.0945" rpy="0 0 0"/>
       <mass value="0.1"/>
-      <inertia ixx="13410" ixy="0.0" ixz="0.0" iyy="13850" iyz="0.0" izz="27150"/>
+      <box_inertia m="0.1" x="${excavatorLenght}" y="${excavatorWidth}" z="${excavatorHeight}"/>
     </inertial>
     <visual>

Commit message: Added transmission to arm joints

File: rover_description/urdf/rover.xacro (robot description, xacro)
@@ -118,4 +118,14 @@
     </collision>
   </link>
+  <transmission name="arm_joint_0_trans">
+    <type>transmission_interface/SimpleTransmission</type>
+    <joint name="arm_joint_0">
+      <hardwareInterface>PositionJointInterface</hardwareInterface>
+    </joint>
+    <actuator name="arm_joint_0_Motor">
+      <hardwareInterface>EffortJointInterface</hardwareInterface>
+      <mechanicalReduction>10</mechanicalReduction>
+    </actuator>
+  </transmission>
   <joint name="joint_base_side_plate" type="fixed">
     <parent link="arm_base_link"/>
@@ -144,4 +154,14 @@
     </collision>
   </link>
+  <transmission name="joint_base_side_plate_trans">
+    <type>transmission_interface/SimpleTransmission</type>
+    <joint name="joint_base_side_plate">
+      <hardwareInterface>PositionJointInterface</hardwareInterface>
+    </joint>
+    <actuator name="arm_joint_0_Motor">
+      <hardwareInterface>EffortJointInterface</hardwareInterface>
+      <mechanicalReduction>10</mechanicalReduction>
+    </actuator>
+  </transmission>
   <joint name="arm_joint_1" type="revolute">
     <parent link="side_plate"/>
@@ -172,4 +192,14 @@
     </inertial>
   </link>
+  <transmission name="arm_link_1_trans">
+    <type>transmission_interface/SimpleTransmission</type>
+    <joint name="arm_link_1">
+      <hardwareInterface>PositionJointInterface</hardwareInterface>
+    </joint>
+    <actuator name="arm_link_1_Motor">
+      <hardwareInterface>EffortJointInterface</hardwareInterface>
+      <mechanicalReduction>10</mechanicalReduction>
+    </actuator>
+  </transmission>
   <joint name="arm_joint_2" type="revolute">
     <parent link="arm_link_1"/>
@@ -200,4 +230,14 @@
     </inertial>
   </link>
+  <transmission name="arm_link_2_trans">
+    <type>transmission_interface/SimpleTransmission</type>
+    <joint name="arm_link_2">
+      <hardwareInterface>PositionJointInterface</hardwareInterface>
+    </joint>
+    <actuator name="arm_link_2_Motor">
+      <hardwareInterface>EffortJointInterface</hardwareInterface>
+      <mechanicalReduction>10</mechanicalReduction>
+    </actuator>
+  </transmission>
   <joint name="arm_joint_3" type="revolute">
     <parent link="arm_link_2"/>
@@ -228,3 +268,13 @@
     </collision>
   </link>
+  <transmission name="arm_link_3_trans">
+    <type>transmission_interface/SimpleTransmission</type>
+    <joint name="arm_link_3">
+      <hardwareInterface>PositionJointInterface</hardwareInterface>
+    </joint>
+    <actuator name="arm_link_3_Motor">
+      <hardwareInterface>EffortJointInterface</hardwareInterface>
+      <mechanicalReduction>10</mechanicalReduction>
+    </actuator>
+  </transmission>
 </robot>
