Commit message: Changed wheel joint parent

File: rover_description/urdf/macros.xacro (robot description, xacro)
@@ -2,11 +2,13 @@
 <robot>
   <macro name="wheel" params="lr tY tX">
+    <joint name="${lr}_wheel_joint" type="continuous">
+      <parent link="base_link"/>
+      <child link="${lr}_wheel"/>
+      <origin xyz="${(wheelPos*tX)} ${tY*wheelWidth/2+tY*chassisWidth/2} ${wheelDrop}" rpy="0 0 0"/>
+      <axis xyz="0 1 0" rpy="0 0 0"/>
+      <!--limit effort="100" velocity="100"/>
+      <joint_properties damping="0.0" friction="0.0"/-->
+    </joint>
     <link name="${lr}_wheel">
-      <collision>
-        <origin xyz="0 0 0" rpy="0 ${PI/2} ${PI/2}"/>
-        <geometry>
-          <cylinder length="${wheelWidth}" radius="${wheelRadius}"/>
-        </geometry>
-      </collision>
       <visual>
         <origin xyz="0 0 0" rpy="0 ${PI/2} ${PI/2}"/>
@@ -16,4 +18,10 @@
         <material name="black"/>
       </visual>
+      <collision>
+        <origin xyz="0 0 0" rpy="0 ${PI/2} ${PI/2}"/>
+        <geometry>
+          <cylinder length="${wheelWidth}" radius="${wheelRadius}"/>
+        </geometry>
+      </collision>
       <inertial>
         <origin xyz="0 0 0" rpy="0 ${PI/2} ${PI/2}"/>
@@ -30,15 +38,9 @@
       <material>Gazebo/Black</material>
     </gazebo>
-    <joint name="${lr}_wheel_joint" type="continuous">
-      <parent link="chassis"/>
-      <child link="${lr}_wheel"/>
-      <origin xyz="${(wheelPos*tX)} ${tY*wheelWidth/2+tY*chassisWidth/2} 0" rpy="0 0 0"/>
-      <axis xyz="0 1 0" rpy="0 0 0"/>
-      <limit effort="100" velocity="100"/>
-      <joint_properties damping="0.0" friction="0.0"/>
-    </joint>
     <transmission name="${lr}_trans">
       <type>transmission_interface/SimpleTransmission</type>
-      <joint name="${lr}_wheel_hinge"/>
+      <joint name="${lr}_wheel_joint">
+        <hardwareInterface>PositionJointInterface</hardwareInterface>
+      </joint>
       <actuator name="${lr}Motor">
         <hardwareInterface>EffortJointInterface</hardwareInterface>
